File: board/fermenticle.sch (KiCad schematic (older format))
At the start: 28 parts, among them IC1 DS2482-100S, J1 1Wire, J3 POWER, P1 DISPLAY, P2 DO0, P6 SD Card, P7 DO 1-3, U1 74hct125d, U2 7805, U3 PHOTON

Commit message: Better layout for v1.1
Parts:
- removed P2: DO0, w_conn_screw:mstba_2,5%2f2-g-5,08, symbol CONN_01X02
- removed P7: DO 1-3, w_conn_screw:mstba_2,5%2f6-g-5,08, symbol CONN_01X06
- added P2: CONN_01X08, w_conn_screw:mstba_2,5%2f8-g-5,08, symbol CONN_01X08
- renumbered LED1 to LED0, LED3 to LED1, LED4 to LED3
Changed lines of the file:
@@
 LIBS:74hct125d
 LIBS:SparkFun
-LIBS:SimpleBrewPiSpark-cache
+LIBS:fermenticle-cache
 EELAYER 25 0
 EELAYER END
@@
 	1    1950 4000
 	1    0    0    -1
-$EndComp
-$Comp
-L CONN_01X02 P2
-U 1 1 56E0F17F
-P 4400 5650
-F 0 "P2" H 4400 5800 50  0000 C CNN
-F 1 "DO0" V 4500 5650 50  0000 C CNN
-F 2 "w_conn_screw:mstba_2,5%2f2-g-5,08" H 4400 5650 50  0001 C CNN
-F 3 "" H 4400 5650 50  0000 C CNN
-	1    4400 5650
-	-1   0    0    1
 $EndComp
 $Comp
@@
 L GND #PWR023
 U 1 1 56E16000
-P 4950 5900
-F 0 "#PWR023" H 4950 5650 50  0001 C CNN
-F 1 "GND" H 4950 5750 50  0000 C CNN
-F 2 "" H 4950 5900 50  0000 C CNN
-F 3 "" H 4950 5900 50  0000 C CNN
-	1    4950 5900
+P 5250 5900
+F 0 "#PWR023" H 5250 5650 50  0001 C CNN
+F 1 "GND" H 5250 5750 50  0000 C CNN
+F 2 "" H 5250 5900 50  0000 C CNN
+F 3 "" H 5250 5900 50  0000 C CNN
+	1    5250 5900
 	1    0    0    -1
 $EndComp
@@
 Text GLabel 5750 6550 1    60   Input ~ 0
 ACT3_5V
+Text GLabel 2650 4000 2    60   Input ~ 0
+ACT0
+Text GLabel 2650 4100 2    60   Input ~ 0
+ACT0_5V
 Text GLabel 2650 4300 2    60   Input ~ 0
-ACT0
+ACT3
 Text GLabel 2650 4400 2    60   Input ~ 0
-ACT0_5V
+ACT3_5V
+Text GLabel 1300 3900 0    60   Input ~ 0
+ACT1
+Text GLabel 1300 4000 0    60   Input ~ 0
+ACT1_5V
 Text GLabel 1300 4200 0    60   Input ~ 0
-ACT3
+ACT2
 Text GLabel 1300 4300 0    60   Input ~ 0
-ACT3_5V
-Text GLabel 2650 4000 2    60   Input ~ 0
-ACT1
-Text GLabel 2650 4100 2    60   Input ~ 0
-ACT1_5V
-Text GLabel 1300 3900 0    60   Input ~ 0
-ACT2
-Text GLabel 1300 4000 0    60   Input ~ 0
 ACT2_5V
 $Comp
@@
 $EndComp
 $Comp
-L LED0603 LED3
+L LED0603 LED1
 U 1 1 56E1E0C6
 P 6350 5650
-F 0 "LED3" V 6150 5500 50  0000 L BNN
+F 0 "LED1" V 6150 5500 50  0000 L BNN
 F 1 "LED" V 6550 5500 50  0000 L BNN
 F 2 "SparkFun:SparkFun-LED-0603" H 6350 5800 50  0001 C CNN
@@
 $EndComp
 $Comp
-L LED0603 LED4
+L LED0603 LED3
 U 1 1 56E1E143
 P 6350 6800
-F 0 "LED4" V 6150 6650 50  0000 L BNN
+F 0 "LED3" V 6150 6650 50  0000 L BNN
 F 1 "LED" V 6550 6650 50  0000 L BNN
 F 2 "SparkFun:SparkFun-LED-0603" H 6350 6950 50  0001 C CNN
@@
 $EndComp
 $Comp
-L LED0603 LED1
+L LED0603 LED0
 U 1 1 56E1E1B2
 P 5250 5650
-F 0 "LED1" V 5050 5500 50  0000 L BNN
+F 0 "LED0" V 5050 5500 50  0000 L BNN
 F 1 "LED" V 5450 5500 50  0000 L BNN
 F 2 "SparkFun:SparkFun-LED-0603" H 5250 5800 50  0001 C CNN
@@
 Wire Wire Line
 	7250 2200 7900 2200
-Wire Wire Line
-	4600 5900 5250 5900
-Wire Wire Line
-	4600 5900 4600 5700
-Connection ~ 4950 5900
-Wire Wire Line
-	4600 5400 4600 5600
-Connection ~ 4600 5500
 Connection ~ 6500 4400
 Wire Wire Line
@@
 Wire Wire Line
 	6350 5500 6300 5500
-Wire Wire Line
-	4800 5500 4600 5500
 Wire Wire Line
 	5200 6650 5250 6650
@@
 	5550 1950 5650 1950
 $Comp
-L CONN_01X06 P7
-U 1 1 5715B0AA
-P 7450 5850
-F 0 "P7" H 7450 6200 50  0000 C CNN
-F 1 "DO 1-3" V 7550 5850 50  0000 C CNN
-F 2 "w_conn_screw:mstba_2,5%2f6-g-5,08" H 7450 5850 50  0001 C CNN
-F 3 "" H 7450 5850 50  0000 C CNN
-	1    7450 5850
-	1    0    0    -1
-$EndComp
-$Comp
 L GND #PWR027
 U 1 1 5715B72C
@@
 Wire Wire Line
 	4600 6650 4600 6550
+Wire Wire Line
+	4600 5400 4600 5500
+Wire Wire Line
+	4600 5500 4800 5500
+$Comp
+L CONN_01X08 P2
+U 1 1 571C57B7
+P 7450 5950
+F 0 "P2" H 7450 6400 50  0000 C CNN
+F 1 "CONN_01X08" V 7550 5950 50  0000 C CNN
+F 2 "w_conn_screw:mstba_2,5%2f8-g-5,08" H 7450 5950 50  0001 C CNN
+F 3 "" H 7450 5950 50  0000 C CNN
+	1    7450 5950
+	1    0    0    -1
+$EndComp
+$Comp
+L GND #PWR030
+U 1 1 571C5BC3
+P 7150 6200
+F 0 "#PWR030" H 7150 5950 50  0001 C CNN
+F 1 "GND" H 7150 6050 50  0000 C CNN
+F 2 "" H 7150 6200 50  0000 C CNN
+F 3 "" H 7150 6200 50  0000 C CNN
+	1    7150 6200
+	0    1    1    0
+$EndComp
+Text GLabel 7150 6300 0    60   Input ~ 0
+ACT0_5V
+Wire Wire Line
+	7150 6200 7250 6200
+Wire Wire Line
+	7150 6300 7250 6300
 $EndSCHEMATC
